Commit message: update

File: src/assets/robots/ri_plus_4438/xmls/urdf/ri_plus_4438.urdf (robot description, URDF)
Before this commit: robot ri_plus_4438, 26 links, 25 joints
Links:
- link FL_calf: geometry collision mesh filename=../assets/FL_calf.STL; visual mesh filename=../assets/FL_calf.STL
- link FL_foot: geometry collision sphere radius=0.02; visual mesh filename=../assets/FL_foot.STL
- link FL_hip: geometry collision mesh filename=../assets/FL_hip.STL; visual mesh filename=../assets/FL_hip.STL
- link FL_thigh: geometry collision mesh filename=../assets/FL_thigh.STL; visual mesh filename=../assets/FL_thigh.STL
- link FR_calf: geometry collision mesh filename=../assets/FR_calf.STL; visual mesh filename=../assets/FR_calf.STL
- link FR_foot: geometry collision sphere radius=0.02; visual mesh filename=../assets/FR_foot.STL
- link FR_hip: geometry collision mesh filename=../assets/FR_hip.STL; visual mesh filename=../assets/FR_hip.STL
- link FR_thigh: geometry collision mesh filename=../assets/FR_thigh.STL; visual mesh filename=../assets/FR_thigh.STL
- link RL_calf: geometry collision mesh filename=../assets/RL_calf.STL; visual mesh filename=../assets/RL_calf.STL
- link RL_foot: geometry collision sphere radius=0.02; visual mesh filename=../assets/RL_foot.STL
- link RL_hip: geometry collision mesh filename=../assets/RL_hip.STL; visual mesh filename=../assets/RL_hip.STL
- link RL_thigh: geometry collision mesh filename=../assets/RL_thigh.STL; visual mesh filename=../assets/RL_thigh.STL
- link RR_calf: geometry collision mesh filename=../assets/RR_calf.STL; visual mesh filename=../assets/RR_calf.STL
- link RR_foot: geometry collision sphere radius=0.02; visual mesh filename=../assets/RR_foot.STL
- link RR_hip: geometry collision mesh filename=../assets/RR_hip.STL; visual mesh filename=../assets/RR_hip.STL
- link RR_thigh: geometry collision mesh filename=../assets/RR_thigh.STL; visual mesh filename=../assets/RR_thigh.STL
- link base_link: geometry collision mesh filename=../assets/base_link.STL; visual mesh filename=../assets/base_link.STL
- link forearm_link: geometry collision mesh filename=../assets/forearm_link.STL; visual mesh filename=../assets/forearm_link.STL
- link gripper_finger_left: geometry collision mesh filename=../assets/gripper_finger_left.STL; visual mesh filename=../assets/gripper_finger_left.STL
- link gripper_finger_right: geometry collision mesh filename=../assets/gripper_finger_right.STL; visual mesh filename=../assets/gripper_finger_right.STL
- link shoulder_link: geometry collision mesh filename=../assets/shoulder_link.STL; visual mesh filename=../assets/shoulder_link.STL
- link upper_arm_link: geometry collision mesh filename=../assets/upper_arm_link.STL; visual mesh filename=../assets/upper_arm_link.STL
- link wrist1_link: geometry collision mesh filename=../assets/wrist1_link.STL; visual mesh filename=../assets/wrist1_link.STL
- link wrist2_link: geometry collision mesh filename=../assets/wrist2_link.STL; visual mesh filename=../assets/wrist2_link.STL
- link wrist3_link: geometry collision mesh filename=../assets/wrist3_link.STL; visual mesh filename=../assets/wrist3_link.STL
- link xlerobot_base_link: geometry collision mesh filename=../assets/xlerobot_base_link.STL; visual mesh filename=../assets/xlerobot_base_link.STL
